File: Hardware/m2_connector.kicad_sch (KiCad schematic)
At the start: 0 parts

Commit message: Constraints for BGA layout
Parts:
- added J1: Bus_M.2_Socket_E, Connector_PCBEdge:M.2_2230-xx-E, symbol Connector:Bus_M.2_Socket_E
Connections:
- new net: J1.1 (GND), J1.18 (GND), J1.33 (GND), J1.39 (GND), J1.45 (GND), J1.51 (GND), J1.57 (GND), J1.63 (GND), J1.69 (GND), J1.7 (GND), J1.75 (GND)
- new net: J1.2 (3.3V), J1.4 (3.3V), J1.72 (3.3V), J1.74 (3.3V)
Changed lines of the file:
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@@
 	(generator_version "10.0")
 	(paper "A4")
+	(symbol
+		(lib_id "Connector:Bus_M.2_Socket_E")
+		(at 76.2 101.6 0)
+		(unit 1)
+		(body_style 1)
+		(exclude_from_sim no)
+		(in_bom yes)
+		(on_board yes)
+		(in_pos_files yes)
+		(dnp no)
+		(fields_autoplaced yes)
+		(property "Reference" "J1"
+			(at 78.3433 50.8 0)
+			(show_name no)
+			(do_not_autoplace no)
+			(effects
+				(font
+					(size 1.27 1.27)
+				)
+				(justify left)
+			)
+		)
+		(property "Value" "Bus_M.2_Socket_E"
+			(at 78.3433 53.34 0)
+			(show_name no)
+			(do_not_autoplace no)
+			(effects
+				(font
+					(size 1.27 1.27)
+				)
+				(justify left)
+			)
+		)
+		(property "Footprint" "Connector_PCBEdge:M.2_2230-xx-E"
+			(at 76.2 74.93 0)
+			(hide yes)
+			(show_name no)
+			(do_not_autoplace no)
+			(effects
+				(font
+					(size 1.27 1.27)
+				)
+			)
+		)
+		(property "Datasheet" "https://web.archive.org/web/20200613074028/http://read.pudn.com/downloads794/doc/project/3133918/PCIe_M.2_Electromechanical_Spec_Rev1.0_Final_11012013_RS_Clean.pdf#page=150"
+			(at 76.2 88.9 0)
+			(hide yes)
+			(show_name no)
+			(do_not_autoplace no)
+			(effects
+				(font
+					(size 1.27 1.27)
+				)
+			)
+		)
+		(property "Description" "M.2 Socket 1-SD Mechanical Key E"
+			(at 76.2 101.6 0)
+			(hide yes)
+			(show_name no)
+			(do_not_autoplace no)
+			(effects
+				(font
+					(size 1.27 1.27)
+				)
+			)
+		)
+		(pin "43"
+		)
+		(pin "53"
+		)
+		(pin "67"
+		)
+		(pin "50"
+		)
+		(pin "71"
+		)
+		(pin "58"
+		)
+		(pin "20"
+		)
+		(pin "12"
+		)
+		(pin "18"
+		)
+		(pin "69"
+		)
+		(pin "54"
+		)
+		(pin "16"
+		)
+		(pin "61"
+		)
+		(pin "48"
+		)
+		(pin "21"
+		)
+		(pin "14"
+		)
+		(pin "70"
+		)
+		(pin "59"
+		)
+		(pin "56"
+		)
+		(pin "74"
+		)
+		(pin "49"
+		)
+		(pin "68"
+		)
+		(pin "73"
+		)
+		(pin "45"
+		)
+		(pin "15"
+		)
+		(pin "55"
+		)
+		(pin "33"
+		)
+		(pin "57"
+		)
+		(pin "36"
+		)
+		(pin "32"
+		)
+		(pin "13"
+		)
+		(pin "72"
+		)
+		(pin "47"
+		)
+		(pin "41"
+		)
+		(pin "65"
+		)
+		(pin "34"
+		)
+		(pin "40"
+		)
+		(pin "60"
+		)
+		(pin "23"
+		)
+		(pin "5"
+		)
+		(pin "2"
+		)
+		(pin "44"
+		)
+		(pin "52"
+		)
+		(pin "17"
+		)
+		(pin "63"
+		)
+		(pin "46"
+		)
+		(pin "64"
+		)
+		(pin "19"
+		)
+		(pin "4"
+		)
+		(pin "6"
+		)
+		(pin "1"
+		)
+		(pin "51"
+		)
+		(pin "42"
+		)
+		(pin "75"
+		)
+		(pin "11"
+		)
+		(pin "10"
+		)
+		(pin "9"
+		)
+		(pin "8"
+		)
+		(pin "7"
+		)
+		(pin "3"
+		)
+		(pin "22"
+		)
+		(pin "39"
+		)
+		(pin "35"
+		)
+		(pin "62"
+		)
+		(pin "66"
+		)
+		(pin "38"
+		)
+		(pin "37"
+		)
+		(instances
+			(project "NotteXCVR"
+				(path "/66cb547b-932d-4f9e-941e-9414e44abcf1/7efd0e01-571a-47c9-afca-84ba246ae436"
+					(reference "J1")
+					(unit 1)
+				)
+			)
+		)
+	)
 )
