File: Hardware/NotteXCVR.kicad_pcb (KiCad board)
At the start: 2 copper layers, 46.4 x 50.8 mm, 23 parts, among them J1 Bus_PCI_Express_x1, J2 GMI-10-2-1.27-G-10, J3 Conn_Coaxial, J4 Conn_Coaxial, J5 Conn_Coaxial, J6 Conn_Coaxial, J7 Conn_Coaxial, J8 Conn_Coaxial, Q1 2N7002, U1 NC7SZ125M5X, U2 XC7A35T-CSG325, U3 FT232H

Commit message: Trying new fanout technology
Parts:
- moved R1 1.04 mm to (84.2, 90.9), turned to 0 degrees
Connections:
- net Net-(J1-PERn0) renamed /PCIE_Edge/EDGE_TX_N
- net Net-(J1-PERp0) renamed /PCIE_Edge/EDGE_TX_P
- net Net-(J1-REFCLK+) renamed /PCIE_Edge/EDGE_REFCLK_P
- net Net-(J1-REFCLK-) renamed /PCIE_Edge/EDGE_REFCLK_N
Routing:
- net PCIE_RX_N: track 0.57 -> 19.5 mm, vias 1 -> 2
- net PCIE_RX_P: track 0.57 -> 19.5 mm, vias 1 -> 2
- net /FPGA_MGT/UFL_CLK_P: track 0.57 -> 13.7 mm, vias 1 -> 0
- net PCIE_REFCLK_N: track 0.57 -> 13.7 mm
- net /FPGA_MGT/UFL_CLK_N: track 0.57 -> 13.5 mm, vias 1 -> 0
- net PCIE_REFCLK_P: track 0.57 -> 13.3 mm
- net PCIE_TX_P: track 0.57 -> 13.1 mm
- net PCIE_TX_N: track 0.57 -> 12.6 mm
- net /PCIE_Edge/EDGE_TX_N: track 0.00 -> 6.24 mm
- net /PCIE_Edge/EDGE_TX_P: track 0.00 -> 6.23 mm
- net /PCIE_Edge/EDGE_REFCLK_P: track 0.00 -> 6.22 mm
- net /PCIE_Edge/EDGE_REFCLK_N: track 0.00 -> 6.22 mm
- net CFG_D4: track 0.57 -> 2.09 mm, vias 1 -> 0
- net GND: track 43.0 -> 43.9 mm
- net PUDC_B: track 0.57 -> 0.00 mm, vias 1 -> 0
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
Commit message: Updated footprint for J2
Routing:
- net GND: track 43.9 -> 50.7 mm, vias 76 -> 92
- net unconnected-(J2-PadD09): track 0.00 -> 0.42 mm, vias 0 -> 1
- net unconnected-(J2-PadD08): track 0.00 -> 0.42 mm, vias 0 -> 1
- net unconnected-(J2-PadD06): track 0.00 -> 0.42 mm, vias 0 -> 1
- net unconnected-(J2-PadD05): track 0.00 -> 0.42 mm, vias 0 -> 1
- net unconnected-(J2-PadD03): track 0.00 -> 0.42 mm, vias 0 -> 1
- net unconnected-(J2-PadD02): track 0.00 -> 0.42 mm, vias 0 -> 1
- net unconnected-(J2-PadC10): track 0.00 -> 0.42 mm, vias 0 -> 1
- net unconnected-(J2-PadC09): track 0.00 -> 0.42 mm, vias 0 -> 1
- net unconnected-(J2-PadC08): track 0.00 -> 0.42 mm, vias 0 -> 1
- net unconnected-(J2-PadC07): track 0.00 -> 0.42 mm, vias 0 -> 1
- net unconnected-(J2-PadC06): track 0.00 -> 0.42 mm, vias 0 -> 1
- net unconnected-(J2-PadC05): track 0.00 -> 0.42 mm, vias 0 -> 1
- net unconnected-(J2-PadC04): track 0.00 -> 0.42 mm, vias 0 -> 1
- net unconnected-(J2-PadC03): track 0.00 -> 0.42 mm, vias 0 -> 1
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