File: Hardware/NotteXCVR.kicad_pcb (KiCad board)
At the start: 2 copper layers, 46.4 x 50.8 mm, 23 parts, among them J1 Bus_PCI_Express_x1, J2 GMI-10-2-1.27-G-10, J3 Conn_Coaxial, J4 Conn_Coaxial, J5 Conn_Coaxial, J6 Conn_Coaxial, J7 Conn_Coaxial, J8 Conn_Coaxial, Q1 2N7002, U1 NC7SZ125M5X, U2 XC7A35T-CSG325, U3 FT232H

Commit message: I gotta find the right regulators
Parts:
- moved J2 24.8 mm to (64.4, 82.1)
- moved R8 16.0 mm to (63.8, 49.8)
- moved Q1 16.0 mm to (67.1, 44.8)
- moved R2 16.0 mm to (60.5, 69.0)
- moved R4 16.0 mm to (70.5, 58.3)
- moved R5 16.0 mm to (70.3, 56.9)
- moved R7 16.0 mm to (71.2, 46.3)
- moved U1 16.0 mm to (67.3, 50.7)
- moved R3 16.0 mm to (70.6, 60.2)
- moved U3 16.0 mm to (62.2, 61.1)
Connections:
- J3 pad 2: Net-(J3-Ext) -> GND
- J4 pad 2: Net-(J3-Ext) -> GND
- J5 pad 2: Net-(J3-Ext) -> GND
- J6 pad 2: Net-(J3-Ext) -> GND
- J7 pad 2: Net-(J3-Ext) -> GND
- J8 pad 2: Net-(J3-Ext) -> GND
Routing:
- net Net-(J1-~{PRSNT1}): track 0.00 -> 32.6 mm, vias 0 -> 1
- net /FPGA_MGT/MGT_UFL_TX_N: track 0.57 -> 12.2 mm, vias 1 -> 2
- net /FPGA_MGT/MGT_UFL_TX_P: track 0.57 -> 12.1 mm, vias 1 -> 2
- net /FPGA_MGT/MGT_UFL_RX_P: track 0.57 -> 10.6 mm, vias 1 -> 2
- net /FPGA_MGT/MGT_UFL_RX_N: track 0.57 -> 10.4 mm, vias 1 -> 2

Commit message: Started breakout
Parts:
- added C5: 0.1uF, Capacitor_SMD:C_0402_1005Metric, F.Cu at (70.8, 49.7)
- moved R4 14.6 mm to (67.2, 72.5)
- moved R5 13.1 mm to (67.3, 69.7)
- moved R3 11.2 mm to (67.2, 70.9), turned to 180 degrees
- moved J2 2.04 mm to (62.4, 82.1), turned to 90 degrees
Connections:
- net +3V3 renamed +2V5
- J2 pad B03: unconnected-(J2-PadB03) -> GND
- J2 pad B06: unconnected-(J2-PadB06) -> GND
- J2 pad B09: unconnected-(J2-PadB09) -> GND
- J2 pad C02: unconnected-(J2-PadC02) -> GND
- J2 pad C05: unconnected-(J2-PadC05) -> GND
- J2 pad C08: unconnected-(J2-PadC08) -> GND
- J2 pad E02: unconnected-(J2-PadE02) -> GND
- J2 pad E05: unconnected-(J2-PadE05) -> GND
- J2 pad E06: unconnected-(J2-PadE06) -> GND
- J2 pad E09: unconnected-(J2-PadE09) -> GND
- J2 pad F02: unconnected-(J2-PadF02) -> GND
- J2 pad F05: unconnected-(J2-PadF05) -> GND
- J2 pad F06: unconnected-(J2-PadF06) -> GND
- J2 pad F09: unconnected-(J2-PadF09) -> GND
- J2 pad H02: unconnected-(J2-PadH02) -> GND
- J2 pad H05: unconnected-(J2-PadH05) -> GND
- J2 pad H08: unconnected-(J2-PadH08) -> GND
- J2 pad I03: unconnected-(J2-PadI03) -> GND
- J2 pad I06: unconnected-(J2-PadI06) -> GND
- J2 pad I09: unconnected-(J2-PadI09) -> GND
- U2 pad C13: unconnected-(U2A-IO_L11N_T1_SRCC_15-PadC13) -> LGA_CLK4_N
- U2 pad D13: unconnected-(U2A-IO_L11P_T1_SRCC_15-PadD13) -> LGA_CLK4_P
- U2 pad D14: unconnected-(U2A-IO_L12N_T1_MRCC_15-PadD14) -> LGA_CLK5_N
- U2 pad D15: unconnected-(U2A-IO_L13N_T2_MRCC_15-PadD15) -> LGA_CLK6_N
- U2 pad D16: unconnected-(U2A-IO_L14N_T2_SRCC_15-PadD16) -> LGA_CLK7_N
- U2 pad E13: unconnected-(U2A-IO_L12P_T1_MRCC_15-PadE13) -> LGA_CLK5_P
- U2 pad E15: unconnected-(U2A-IO_L13P_T2_MRCC_15-PadE15) -> LGA_CLK6_P
- U2 pad E16: unconnected-(U2A-IO_L14P_T2_SRCC_15-PadE16) -> LGA_CLK7_P
Routing:
- net /FPGA_Config/TCK: track 0.57 -> 11.0 mm, vias 1 -> 2
- net CCLK: track 0.57 -> 10.6 mm, vias 1 -> 2
- net GND: track 50.7 -> 59.1 mm, vias 92 -> 112
- net MODE2: track 0.57 -> 8.40 mm, vias 1 -> 2
- net /FPGA_Config/FPGA_TDI: track 0.57 -> 7.35 mm
- net INIT_B: track 0.57 -> 6.99 mm
- net MODE1: track 0.57 -> 6.81 mm
- net /FPGA_Config/TMS: track 0.57 -> 6.35 mm
- net MODE0: track 0.57 -> 5.93 mm
- net LGA_CLK5_P: track 0.00 -> 4.56 mm, vias 0 -> 1
- net LGA_CLK4_P: track 0.00 -> 4.16 mm, vias 0 -> 1
- net LGA_CLK6_N: track 0.00 -> 4.15 mm, vias 0 -> 1
- net LGA_CLK6_P: track 0.00 -> 4.07 mm, vias 0 -> 1
- net PROG_B: track 0.57 -> 4.60 mm
- net LGA_CLK5_N: track 0.00 -> 3.75 mm, vias 0 -> 1
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