File: Hardware/fpga_gpio.kicad_sch (KiCad schematic)
At the start: 0 parts

Commit message: Constraints for BGA layout
Parts:
- added U1: XC7A50T-CPG236, Package_BGA:Xilinx_CPG236, symbol FPGA_Xilinx_Artix7:XC7A50T-CPG236

Commit message: CSG325?
Parts:
- removed U1: XC7A50T-CPG236, Package_BGA:Xilinx_CPG236, symbol FPGA_Xilinx_Artix7:XC7A50T-CPG236
- added U2: XC7A35T-CSG325, Package_BGA:Xilinx_CSG325, symbol FPGA_Xilinx_Artix7:XC7A35T-CSG325

Commit message: Found the global labels
Connections:
- net at U2.L6 (VCCO_34): now also U2.M3 (VCCO_34), U2.P7 (VCCO_34), U2.R4 (VCCO_34), U2.T1 (VCCO_34), U2.V5 (VCCO_34)
Changed lines of the file:
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@@
 	(generator_version "10.0")
 	(paper "B")
+	(junction
+		(at 187.96 45.72)
+		(diameter 0)
+		(color 0 0 0 0)
+	)
+	(junction
+		(at 182.88 45.72)
+		(diameter 0)
+		(color 0 0 0 0)
+	)
+	(junction
+		(at 185.42 45.72)
+		(diameter 0)
+		(color 0 0 0 0)
+	)
+	(junction
+		(at 180.34 45.72)
+		(diameter 0)
+		(color 0 0 0 0)
+	)
+	(wire
+		(pts
+			(xy 185.42 45.72) (xy 187.96 45.72)
+		)
+		(stroke
+			(width 0)
+			(type default)
+		)
+	)
+	(wire
+		(pts
+			(xy 180.34 45.72) (xy 182.88 45.72)
+		)
+		(stroke
+			(width 0)
+			(type default)
+		)
+	)
+	(wire
+		(pts
+			(xy 177.8 45.72) (xy 180.34 45.72)
+		)
+		(stroke
+			(width 0)
+			(type default)
+		)
+	)
+	(wire
+		(pts
+			(xy 187.96 45.72) (xy 190.5 45.72)
+		)
+		(stroke
+			(width 0)
+			(type default)
+		)
+	)
+	(wire
+		(pts
+			(xy 182.88 45.72) (xy 185.42 45.72)
+		)
+		(stroke
+			(width 0)
+			(type default)
+		)
+	)
 	(symbol
 		(lib_id "FPGA_Xilinx_Artix7:XC7A35T-CSG325")

Commit message: I gotta find the right regulators
Changed lines of the file:
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@@
+	(wire
+		(pts
+			(xy 146.05 127) (xy 167.64 127)
+		)
+		(stroke
+			(width 0)
+			(type default)
+		)
+	)
+	(wire
+		(pts
+			(xy 146.05 119.38) (xy 167.64 119.38)
+		)
+		(stroke
+			(width 0)
+			(type default)
+		)
+	)
 	(wire
 		(pts
@@
 	(wire
 		(pts
+			(xy 146.05 121.92) (xy 167.64 121.92)
+		)
+		(stroke
+			(width 0)
+			(type default)
+		)
+	)
+	(wire
+		(pts
+			(xy 146.05 124.46) (xy 167.64 124.46)
+		)
+		(stroke
+			(width 0)
+			(type default)
+		)
+	)
+	(wire
+		(pts
 			(xy 177.8 45.72) (xy 180.34 45.72)
+		)
+		(stroke
+			(width 0)
+			(type default)
+		)
+	)
+	(wire
+		(pts
+			(xy 146.05 137.16) (xy 167.64 137.16)
 		)
 		(stroke
@@
 	(wire
 		(pts
+			(xy 146.05 129.54) (xy 167.64 129.54)
+		)
+		(stroke
+			(width 0)
+			(type default)
+		)
+	)
+	(wire
+		(pts
+			(xy 146.05 132.08) (xy 167.64 132.08)
+		)
+		(stroke
+			(width 0)
+			(type default)
+		)
+	)
+	(wire
+		(pts
 			(xy 182.88 45.72) (xy 185.42 45.72)
 		)
 		(stroke
+			(width 0)
+			(type default)
+		)
+	)
+	(wire
+		(pts
+			(xy 146.05 134.62) (xy 167.64 134.62)
+		)
+		(stroke
