File: Hardware/off_board_interface.kicad_sch (KiCad schematic)
At the start: 1 part, among them J2 GMI-10-2-1.27-G-10

Commit message: Found the global labels
Connections:
- net GND: now reaches J2.J01
- net GND: now also J2.A01, J2.A04, J2.A07, J2.A10, J2.D01, J2.D04, J2.D07, J2.D10, J2.G01, J2.G04, J2.G07, J2.G10, J2.J04, J2.J07, J2.J10

Commit message: Started breakout
Connections:
- net GND: now also J2.B03, J2.B06, J2.B09, J2.C02, J2.C05, J2.C08, J2.E02, J2.E05, J2.E06, J2.E09, J2.F02, J2.F05, J2.F06, J2.F09, J2.H02, J2.H05, J2.H08, J2.I03, J2.I06, J2.I09
