File: Hardware/_restore_backup_2026-07-31T22-59-24-820/NotteXCVR.kicad_pcb (KiCad board)
At the start: 2 copper layers, 46.4 x 50.8 mm, 23 parts, among them J1 Bus_PCI_Express_x1, J2 GMI-10-2-1.27-G-10, J3 Conn_Coaxial, J4 Conn_Coaxial, J5 Conn_Coaxial, J6 Conn_Coaxial, J7 Conn_Coaxial, J8 Conn_Coaxial, Q1 2N7002, U1 NC7SZ125M5X, U2 XC7A35T-CSG325, U3 FT232H

Commit message: Configuration interface, reducing trace width/space
Parts:
- removed Q1: 2N7002, Package_TO_SOT_SMD:SOT-23
- removed R2: 100, Resistor_SMD:R_0402_1005Metric
- removed R3: 1k, Resistor_SMD:R_0402_1005Metric
- removed R4, R5, R7, R8: 4.7k, Resistor_SMD:R_0402_1005Metric
- removed U1: NC7SZ125M5X, Package_TO_SOT_SMD:SOT-23-5
- removed U3: FT232H, Package_QFP:LQFP-48_7x7mm_P0.5mm
- moved J2 7.39 mm to (86.8, 58.9)
Connections:
- U2 pad A16: +3V3 -> Net-(U2A-VCCO_15-PadA16)
- U2 pad B13: +3V3 -> Net-(U2A-VCCO_15-PadA16)
- U2 pad C10: +3V3 -> Net-(U2A-VCCO_15-PadA16)
- U2 pad D17: +3V3 -> Net-(U2A-VCCO_15-PadA16)
- U2 pad E10: +3V3 -> unconnected-(U2E-VCCO_0-PadE10)
- U2 pad E12: +3V3 -> unconnected-(U2E-CFGBVS_0-PadE12)
- U2 pad E14: +3V3 -> Net-(U2A-VCCO_15-PadA16)
- U2 pad E8: CCLK -> unconnected-(U2E-CCLK_0-PadE8)
- U2 pad F12: DONE -> unconnected-(U2E-DONE_0-PadF12)
- U2 pad F13: MODE2 -> unconnected-(U2E-M2_0-PadF13)
- U2 pad F8: /FPGA_Config/TCK -> unconnected-(U2E-TCK_0-PadF8)
- U2 pad G18: +3V3 -> Net-(U2A-VCCO_15-PadA16)
- U2 pad H15: +3V3 -> Net-(U2A-VCCO_15-PadA16)
- U2 pad J14: CFG_D6 -> unconnected-(U2A-IO_L5P_T0_D06_14-PadJ14)
- U2 pad J15: CFG_D2 -> unconnected-(U2A-IO_L2P_T0_D02_14-PadJ15)
- U2 pad J16: CFG_D3 -> unconnected-(U2A-IO_L2N_T0_D03_14-PadJ16)
- U2 pad J18: PUDC_B -> unconnected-(U2A-IO_L3P_T0_DQS_PUDC_B_14-PadJ18)
- U2 pad K15: CFG_D7 -> unconnected-(U2A-IO_L5N_T0_D07_14-PadK15)
- U2 pad K16: CFG_D0 -> unconnected-(U2A-IO_L1P_T0_D00_MOSI_14-PadK16)
- U2 pad K17: CFG_D4 -> unconnected-(U2A-IO_L4P_T0_D04_14-PadK17)
- U2 pad K18: CFG_EMCCLK -> unconnected-(U2A-IO_L3N_T0_DQS_EMCCLK_14-PadK18)
- U2 pad L15: CFG_CS -> unconnected-(U2A-IO_L6P_T0_FCS_B_14-PadL15)
- U2 pad L16: +3V3 -> Net-(U2A-VCCO_14-PadL16)
- U2 pad L17: CFG_D1 -> unconnected-(U2A-IO_L1N_T0_D01_DIN_14-PadL17)
- U2 pad L18: CFG_D5 -> unconnected-(U2A-IO_L4N_T0_D05_14-PadL18)
- U2 pad P10: PROG_B -> unconnected-(U2E-PROGRAM_B_0-PadP10)
- U2 pad P14: LGA_CLK1_P -> unconnected-(U2A-IO_L12P_T1_MRCC_14-PadP14)
- U2 pad P15: LGA_CLK0_P -> unconnected-(U2A-IO_L11P_T1_SRCC_14-PadP15)
- U2 pad P16: LGA_CLK0_N -> unconnected-(U2A-IO_L11N_T1_SRCC_14-PadP16)
- U2 pad P17: +3V3 -> Net-(U2A-VCCO_14-PadL16)
- U2 pad R10: +3V3 -> unconnected-(U2E-VCCO_0-PadR10)
- U2 pad R11: MODE1 -> unconnected-(U2E-M1_0-PadR11)
- U2 pad R12: MODE0 -> unconnected-(U2E-M0_0-PadR12)
- U2 pad R14: +3V3 -> Net-(U2A-VCCO_14-PadL16)
- U2 pad R15: LGA_CLK1_N -> unconnected-(U2A-IO_L12N_T1_MRCC_14-PadR15)
- U2 pad R16: LGA_CLK3_P -> unconnected-(U2A-IO_L14P_T2_SRCC_14-PadR16)
- U2 pad R17: LGA_CLK3_N -> unconnected-(U2A-IO_L14N_T2_SRCC_14-PadR17)
- U2 pad R18: CFG_RDWR -> unconnected-(U2A-IO_L15P_T2_DQS_RDWR_B_14-PadR18)
- U2 pad R8: /FPGA_Config/TMS -> unconnected-(U2E-TMS_0-PadR8)
- U2 pad T10: INIT_B -> unconnected-(U2E-INIT_B_0-PadT10)
- U2 pad T11: +3V3 -> Net-(U2A-VCCO_14-PadL16)
- U2 pad T14: LGA_CLK2_P -> unconnected-(U2A-IO_L13P_T2_MRCC_14-PadT14)
- U2 pad T15: LGA_CLK2_N -> unconnected-(U2A-IO_L13N_T2_MRCC_14-PadT15)
- U2 pad T17: CFG_CSI -> unconnected-(U2A-IO_L16P_T2_CSI_B_14-PadT17)
- U2 pad T18: CFG_DOUT -> unconnected-(U2A-IO_L15N_T2_DQS_DOUT_CSO_B_14-PadT18)
- U2 pad T8: /FPGA_Config/FPGA_TDO_LGA_TDI -> unconnected-(U2E-TDO_0-PadT8)
- U2 pad T9: /FPGA_Config/FPGA_TDI -> unconnected-(U2E-TDI_0-PadT9)
- U2 pad U18: +3V3 -> Net-(U2A-VCCO_14-PadL16)
- U2 pad U8: +3V3 -> Net-(U2A-VCCO_14-PadL16)
- U2 pad V15: +3V3 -> Net-(U2A-VCCO_14-PadL16)
Routing:
- net +3V3: track 9.62 -> 0.00 mm, vias 17 -> 0
- net Net-(U2A-VCCO_14-PadL16): track 0.00 -> 3.96 mm, vias 0 -> 7
- net Net-(U2A-VCCO_15-PadA16): track 0.00 -> 3.96 mm, vias 0 -> 7
- net LGA_CLK2_P: track 0.59 -> 0.00 mm, vias 1 -> 0
- net CFG_D3: track 0.57 -> 0.00 mm, vias 1 -> 0
- net unconnected-(U2E-TDI_0-PadT9): track 0.00 -> 0.57 mm, vias 0 -> 1
- net unconnected-(U2E-M1_0-PadR11): track 0.00 -> 0.57 mm, vias 0 -> 1
- net unconnected-(U2E-M0_0-PadR12): track 0.00 -> 0.57 mm, vias 0 -> 1
- net unconnected-(U2E-CFGBVS_0-PadE12): track 0.00 -> 0.57 mm, vias 0 -> 1
- net unconnected-(U2A-IO_L4P_T0_D04_14-PadK17): track 0.00 -> 0.57 mm, vias 0 -> 1
- net unconnected-(U2A-IO_L4N_T0_D05_14-PadL18): track 0.00 -> 0.57 mm, vias 0 -> 1
- net unconnected-(U2A-IO_L3P_T0_DQS_PUDC_B_14-PadJ18): track 0.00 -> 0.57 mm, vias 0 -> 1
- net unconnected-(U2A-IO_L3N_T0_DQS_EMCCLK_14-PadK18): track 0.00 -> 0.57 mm, vias 0 -> 1
- net unconnected-(U2A-IO_L2N_T0_D03_14-PadJ16): track 0.00 -> 0.57 mm, vias 0 -> 1
- net unconnected-(U2A-IO_L1P_T0_D00_MOSI_14-PadK16): track 0.00 -> 0.57 mm, vias 0 -> 1
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